File: hw/singleGates/1-BitSelect.brd (EAGLE design)
At the start: 12 x 15 mm, 15 parts, among them Q1 BC817, Q2 BC817, Q3 BC817, Q4 BC817, Q5 BC817, Q6 BC817

Commit message: Updated supply line names to be more spice compatible
Connections:
- net V+ renamed _VP
- net V- renamed _VN
Changed lines of the file:
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@@
 <?xml version="1.0" encoding="utf-8"?>
 <!DOCTYPE eagle SYSTEM "eagle.dtd">
-<eagle version="7.4.0">
+<eagle version="7.3.0">
 <drawing>
 <settings>
@@
 </elements>
 <signals>
-<signal name="V-">
+<signal name="_VN">
 <wire x1="7.45" y1="7.6" x2="7.5" y2="7.8" width="0.2" layer="1"/>
 <wire x1="3.05" y1="7.6" x2="3.4" y2="7.6" width="0.2" layer="1"/>
@@
 <contactref element="Q3" pad="P$1"/>
 </signal>
-<signal name="V+">
+<signal name="_VP">
 <contactref element="R4" pad="2"/>
 <contactref element="R1" pad="2"/>
