File: hw/singleGates/1-BitSelect.brd (EAGLE design)
At the start: 12 x 15 mm, 15 parts, among them Q1 BC817, Q2 BC817, Q3 BC817, Q4 BC817, Q5 BC817, Q6 BC817

Commit message: Removed dimension border, added tPlace border
Other:
- board outline removed

Commit message: Made components to only have connections on 2 sides
Routing:
- net A: track 1.82 -> 4.29 mm
- net SEL: track 5.87 -> 4.93 mm
Changed lines of the file:
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@@
 <setting verticaltext="up"/>
 </settings>
-<grid distance="0.5" unitdist="mm" unit="mm" style="lines" multiple="1" display="yes" altdistance="0.25" altunitdist="mm" altunit="mm"/>
+<grid distance="0.1" unitdist="mm" unit="mm" style="lines" multiple="1" display="yes" altdistance="0.05" altunitdist="mm" altunit="mm"/>
 <layers>
 <layer number="1" name="Top" color="4" fill="1" visible="yes" active="yes"/>
@@
 <contactref element="R2" pad="1"/>
 <contactref element="R5" pad="1"/>
-<wire x1="0" y1="1" x2="1.9" y2="1" width="0.2" layer="1"/>
-<wire x1="1.9" y1="1" x2="2.3" y2="1.4" width="0.2" layer="1"/>
+<wire x1="2" y1="0" x2="2" y2="1.1" width="0.2" layer="1"/>
+<wire x1="2" y1="1.1" x2="2.3" y2="1.4" width="0.2" layer="1"/>
 <wire x1="2.3" y1="1.4" x2="2.3" y2="2.3" width="0.2" layer="1"/>
 <wire x1="2.3" y1="2.3" x2="2.5" y2="2.5" width="0.2" layer="1"/>
@@
 <signal name="A">
 <contactref element="R3" pad="1"/>
-<wire x1="1" y1="3.4" x2="1" y2="4.05" width="0.2" layer="1"/>
-<wire x1="0.6" y1="3" x2="0" y2="3" width="0.2" layer="1" style="shortdash"/>
-<wire x1="0.6" y1="3" x2="1" y2="3.4" width="0.2" layer="1"/>
+<wire x1="1" y1="4" x2="1" y2="4.05" width="0.2" layer="1"/>
+<wire x1="1" y1="3.9" x2="0.9" y2="3.9" width="0.2" layer="1"/>
+<wire x1="0.9" y1="3.9" x2="1" y2="3.9" width="0.2" layer="1"/>
+<wire x1="1" y1="3.9" x2="1" y2="0" width="0.2" layer="1"/>
+<wire x1="1" y1="4" x2="0.9" y2="3.9" width="0.2" layer="1"/>
 </signal>
 <signal name="B">
 <contactref element="R7" pad="1"/>
-<wire x1="0" y1="2" x2="1.6" y2="2" width="0.2" layer="1"/>
-<wire x1="1.6" y1="2" x2="1.9" y2="2.3" width="0.2" layer="1"/>
+<wire x1="1.5" y1="0" x2="1.5" y2="1.9" width="0.2" layer="1"/>
 <wire x1="1.9" y1="2.3" x2="1.9" y2="4.5" width="0.2" layer="1"/>
 <wire x1="1.9" y1="4.5" x2="2.3" y2="4.9" width="0.2" layer="1"/>
@@
 <wire x1="4.4" y1="4" x2="5.45" y2="4" width="0.2" layer="1"/>
 <wire x1="5.45" y1="4" x2="5.5" y2="4.05" width="0.2" layer="1"/>
+<wire x1="1.5" y1="1.9" x2="1.9" y2="2.3" width="0.2" layer="1"/>
 </signal>
 <signal name="I-S2">

Commit message: Fixing stuff
Changed lines of the file:
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@@
 <?xml version="1.0" encoding="utf-8"?>
 <!DOCTYPE eagle SYSTEM "eagle.dtd">
-<eagle version="7.4.0">
+<eagle version="7.3.0">
 <drawing>
 <settings>
@@
 <wire x1="10.1" y1="12.5" x2="10.4" y2="12.8" width="0.2" layer="1"/>
 <wire x1="10.4" y1="12.8" x2="10.95" y2="12.8" width="0.2" layer="1"/>
-<wire x1="11" y1="0" x2="11" y2="0.8" width="0.2" layer="1" style="shortdash"/>
+<wire x1="11" y1="0" x2="11" y2="0.8" width="0.2" layer="1"/>
 <wire x1="11" y1="0.8" x2="11" y2="1.2" width="0.2" layer="1"/>
 <wire x1="11" y1="1.2" x2="11.2" y2="1.4" width="0.2" layer="1"/>
