File: hw/singleGates/1-BitSelect.sch (EAGLE design)
At the start: 15 parts, among them Q1 BC817, Q2 BC817, Q3 BC817, Q4 BC817, Q5 BC817, Q6 BC817

Commit message: Updated supply line names to be more spice compatible
Connections:
- net V+ renamed _VP
- net V- renamed _VN
Other:
- note removed: "1-BIT SELECT"
Changed lines of the file:
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@@
 <?xml version="1.0" encoding="utf-8"?>
 <!DOCTYPE eagle SYSTEM "eagle.dtd">
-<eagle version="7.4.0">
+<eagle version="7.3.0">
 <drawing>
 <settings>
@@
 <wire x1="-30.48" y1="33.02" x2="-30.48" y2="-33.02" width="0.4064" layer="97" style="longdash"/>
 <wire x1="-30.48" y1="-33.02" x2="30.48" y2="-33.02" width="0.4064" layer="97" style="longdash"/>
-<text x="208.28" y="86.36" size="2.54" layer="97" ratio="12">1-BIT SELECT</text>
 <wire x1="30.48" y1="33.02" x2="30.48" y2="-33.02" width="0.4064" layer="97" style="longdash"/>
 </plain>
@@
 </busses>
 <nets>
-<net name="V-" class="0">
+<net name="_VN" class="0">
 <segment>
 <pinref part="Q2" gate="G$1" pin="EMITTER"/>
@@
 </segment>
 </net>
-<net name="V+" class="0">
+<net name="_VP" class="0">
 <segment>
 <pinref part="R4" gate="G$1" pin="2"/>
