File: hw/singleGates/1-BitSelect.sch (EAGLE design)
At the start: 15 parts, among them Q1 BC817, Q2 BC817, Q3 BC817, Q4 BC817, Q5 BC817, Q6 BC817

Commit message: Basic cleanups
Other:
- moved on the sheet: Q1, Q2, Q3, Q4, Q5, Q6, R1, R2, R3, R4, R5, R6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
