File: hw/singleGates/3-BitSelect.brd (EAGLE design)
At the start: 36 parts, among them Q1 BC817, Q10 BC817, Q11 BC817, Q12 BC817, Q13 BC817, Q14 BC817, Q15 BC817, Q16 BC817, Q17 BC817, Q2 BC817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

Commit message: Updated supply line names to be more spice compatible
Connections:
- net V+ renamed _VP
- net V- renamed _VN
Changed lines of the file:
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@@
 <?xml version="1.0" encoding="utf-8"?>
 <!DOCTYPE eagle SYSTEM "eagle.dtd">
-<eagle version="7.4.0">
+<eagle version="7.3.0">
 <drawing>
 <settings>
@@
 </elements>
 <signals>
-<signal name="V-">
+<signal name="_VN">
 <wire x1="3.25" y1="5.1" x2="3.25" y2="5.15" width="0.2" layer="1"/>
 <wire x1="3.25" y1="5.15" x2="3.3" y2="5.2" width="0.2" layer="1"/>
@@
 <wire x1="20.9" y1="5.1" x2="20.85" y2="5.1" width="0" layer="19" extent="1-1"/>
 </signal>
-<signal name="V+">
+<signal name="_VP">
 <contactref element="R1" pad="2"/>
 <contactref element="R19" pad="2"/>
