File: hw/singleGates/3-BitSelect.sch (EAGLE design)
At the start: 36 parts, among them Q1 BC817, Q10 BC817, Q11 BC817, Q12 BC817, Q13 BC817, Q14 BC817, Q15 BC817, Q16 BC817, Q17 BC817, Q2 BC817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

Commit message: Updated supply line names to be more spice compatible
Connections:
- net V+ renamed _VP
- net V- renamed _VN
Changed lines of the file:
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@@
 <?xml version="1.0" encoding="utf-8"?>
 <!DOCTYPE eagle SYSTEM "eagle.dtd">
-<eagle version="7.4.0">
+<eagle version="7.3.0">
 <drawing>
 <settings>
@@
 </busses>
 <nets>
-<net name="V-" class="0">
+<net name="_VN" class="0">
 <segment>
 <pinref part="Q2" gate="G$1" pin="EMITTER"/>
@@
 </segment>
 </net>
-<net name="V+" class="0">
+<net name="_VP" class="0">
 <segment>
 <pinref part="R1" gate="G$1" pin="2"/>
