File: hw/singleGates/NAND.brd (EAGLE design)
At the start: 5 parts, among them Q1 BC817, Q2 BC817

Commit message: Updated supply line names to be more spice compatible
Connections:
- net V+ renamed _VP
- net V- renamed _VN
Changed lines of the file:
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@@
 <?xml version="1.0" encoding="utf-8"?>
 <!DOCTYPE eagle SYSTEM "eagle.dtd">
-<eagle version="7.4.0">
+<eagle version="7.3.0">
 <drawing>
 <settings>
@@
 <contactref element="Q2" pad="P$3"/>
 </signal>
-<signal name="V+">
+<signal name="_VP">
 <contactref element="R3" pad="2"/>
 <wire x1="2.75" y1="7.45" x2="2.8" y2="7.5" width="0.2" layer="1"/>
@@
 <wire x1="2.75" y1="7.45" x2="2.75" y2="7.4" width="0" layer="19" extent="1-1"/>
 </signal>
-<signal name="V-">
+<signal name="_VN">
 <contactref element="Q2" pad="P$2"/>
 <wire x1="6" y1="6.6" x2="6" y2="8.5" width="0.2" layer="1"/>
