File: hw/singleGates/NOT-A.brd (EAGLE design)
At the start: 3 parts, among them Q1 BC817

Commit message: Updated supply line names to be more spice compatible
Connections:
- net V+ renamed _VP
- net V- renamed _VN
Changed lines of the file:
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@@
 <?xml version="1.0" encoding="utf-8"?>
 <!DOCTYPE eagle SYSTEM "eagle.dtd">
-<eagle version="7.4.0">
+<eagle version="7.3.0">
 <drawing>
 <settings>
@@
 </elements>
 <signals>
-<signal name="V-">
+<signal name="_VN">
 <wire x1="2.95" y1="3.2" x2="2.95" y2="6.15" width="0.2" layer="1"/>
 <wire x1="2.95" y1="6.15" x2="2.7" y2="6.4" width="0.2" layer="1"/>
@@
 <wire x1="3" y1="1.15" x2="2.85" y2="1.3" width="0.2" layer="1"/>
 </signal>
-<signal name="V+">
+<signal name="_VP">
 <contactref element="R2" pad="1"/>
 <wire x1="3" y1="8.5" x2="3" y2="8.4" width="0.2" layer="1"/>
