File: hw/singleGates/OR.brd (EAGLE design)
At the start: 7.1 x 12.5 mm, 8 parts, among them Q1 BC817, Q2 BC817, Q3 BC817

Commit message: Updated supply line names to be more spice compatible
Connections:
- net V+ renamed _VP
- net V- renamed _VN
Changed lines of the file:
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@@
 <?xml version="1.0" encoding="utf-8"?>
 <!DOCTYPE eagle SYSTEM "eagle.dtd">
-<eagle version="7.4.0">
+<eagle version="7.3.0">
 <drawing>
 <settings>
@@
 <contactref element="Q3" pad="P$3"/>
 </signal>
-<signal name="V-">
+<signal name="_VN">
 <wire x1="2.85" y1="3.3" x2="2.85" y2="4.15" width="0.2" layer="1"/>
 <wire x1="2.85" y1="4.15" x2="3.1" y2="4.4" width="0.2" layer="1"/>
@@
 <contactref element="Q3" pad="P$2"/>
 </signal>
-<signal name="V+">
+<signal name="_VP">
 <contactref element="R5" pad="2"/>
 <contactref element="R3" pad="2"/>
