File: hw/singleGates/XOR.brd (EAGLE design)
At the start: 15 parts, among them Q1 BC817, Q2 BC817, Q3 BC817, Q4 BC817, Q5 BC817, Q6 BC817

Commit message: Updated supply line names to be more spice compatible
Connections:
- net V+ renamed _VP
- net V- renamed _VN
Changed lines of the file:
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@@
 <?xml version="1.0" encoding="utf-8"?>
 <!DOCTYPE eagle SYSTEM "eagle.dtd">
-<eagle version="7.4.0">
+<eagle version="7.3.0">
 <drawing>
 <settings>
@@
 </elements>
 <signals>
-<signal name="V-">
+<signal name="_VN">
 <contactref element="R3" pad="1"/>
 <wire x1="8.4" y1="1.95" x2="8.4" y2="2.6" width="0.2" layer="1"/>
@@
 <contactref element="Q6" pad="P$2"/>
 </signal>
-<signal name="V+">
+<signal name="_VP">
 <contactref element="R9" pad="2"/>
 <wire x1="1.1" y1="9.7" x2="1.1" y2="11" width="0.2" layer="1"/>

Commit message: XOR tests
Parts:
- R3, R6: value 10k -> 1k
Changed lines of the file:
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@@
 <?xml version="1.0" encoding="utf-8"?>
 <!DOCTYPE eagle SYSTEM "eagle.dtd">
-<eagle version="7.3.0">
+<eagle version="7.4.0">
 <drawing>
 <settings>
@@
 <attribute name="SV_SPICE_PREFIX" value="R" x="6" y="2.8" size="1.778" layer="27" rot="R90" display="off"/>
 </element>
-<element name="R3" library="p.peter-gator" package="R0603" value="10k" x="8.4" y="2.8" smashed="yes" rot="R90">
+<element name="R3" library="p.peter-gator" package="R0603" value="1k" x="8.4" y="2.8" smashed="yes" rot="R90">
 <attribute name="SV_SPICE_ORDER" value="1;2" x="8.4" y="2.8" size="1.778" layer="27" rot="R90" display="off"/>
 <attribute name="SV_SPICE_PREFIX" value="R" x="8.4" y="2.8" size="1.778" layer="27" rot="R90" display="off"/>
 </element>
-<element name="R6" library="p.peter-gator" package="R0603" value="10k" x="2" y="9.7" smashed="yes" rot="R180">
+<element name="R6" library="p.peter-gator" package="R0603" value="1k" x="2" y="9.7" smashed="yes" rot="R180">
 <attribute name="SV_SPICE_ORDER" value="1;2" x="2" y="9.7" size="1.778" layer="27" rot="R180" display="off"/>
 <attribute name="SV_SPICE_PREFIX" value="R" x="2" y="9.7" size="1.778" layer="27" rot="R180" display="off"/>
