File: hw/singleGates/XOR.sch (EAGLE design)
At the start: 15 parts, among them Q1 BC817, Q2 BC817, Q3 BC817, Q4 BC817, Q5 BC817, Q6 BC817

Commit message: Basic cleanups
Changed lines of the file:
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@@
 <wire x1="-10.16" y1="-27.94" x2="-10.16" y2="-30.48" width="0.1524" layer="91"/>
 <junction x="-10.16" y="-27.94"/>
-<label x="-12.7" y="-27.94" size="1.778" layer="95"/>
 <wire x1="5.08" y1="-5.08" x2="5.08" y2="-2.54" width="0.1524" layer="91"/>
 <wire x1="7.62" y1="-5.08" x2="5.08" y2="-5.08" width="0.1524" layer="91"/>
@@
 <pinref part="R7" gate="G$1" pin="1"/>
 <wire x1="17.78" y1="2.54" x2="10.16" y2="2.54" width="0.1524" layer="91"/>
-<label x="38.1" y="25.4" size="1.778" layer="95"/>
 <pinref part="Q3" gate="G$1" pin="COLLECTOR"/>
 <pinref part="Q4" gate="G$1" pin="COLLECTOR"/>
@@
 <wire x1="38.1" y1="10.16" x2="38.1" y2="0" width="0.1524" layer="91"/>
 <wire x1="38.1" y1="0" x2="43.18" y2="0" width="0.1524" layer="91"/>
-<label x="38.1" y="0" size="1.778" layer="95"/>
 <junction x="38.1" y="0"/>
 <pinref part="Q5" gate="G$1" pin="COLLECTOR"/>
@@
 <wire x1="-45.72" y1="22.86" x2="-45.72" y2="17.78" width="0.1524" layer="91"/>
 <junction x="-45.72" y="17.78"/>
-<label x="-47.752" y="15.24" size="1.778" layer="95"/>
 </segment>
 </net>
@@
 <pinref part="R5" gate="G$1" pin="1"/>
 <wire x1="-15.24" y1="-15.24" x2="-12.7" y2="-15.24" width="0.1524" layer="91"/>
-<label x="-47.498" y="-19.812" size="1.778" layer="95"/>
 <junction x="-45.72" y="-7.62"/>
 </segment>
@@
 <pinref part="R8" gate="G$1" pin="1"/>
 <wire x1="15.24" y1="-15.24" x2="17.78" y2="-15.24" width="0.1524" layer="91"/>
-<label x="38.1" y="-25.4" size="1.778" layer="95"/>
 <pinref part="Q2" gate="G$1" pin="EMITTER"/>
 </segment>
@@
 <wire x1="-10.16" y1="27.94" x2="-10.16" y2="30.48" width="0.1524" layer="91"/>
 <junction x="-10.16" y="27.94"/>
-<label x="-7.62" y="27.94" size="1.778" layer="95"/>
 <pinref part="R6" gate="G$1" pin="2"/>
 <wire x1="5.08" y1="27.94" x2="5.08" y2="22.86" width="0.1524" layer="91"/>
