File: hw/composites/alu_slice.sch (EAGLE design)
At the start: 13 parts

Commit message: Trying to mimize gates some more
Parts:
- CON2: value (none) -> GENERIC-2X10
Connections:
- net +5V: now also NAND1.V+, NOT1.V+, NOT2.V+, OR1.V+, OR3.V+, SEL1.V+, SEL2.V+, SEL3.V+, XOR1.V+, XOR2.V+, XOR3.V+, XOR4.V+; no longer NAND1._VP, NOT1._VP, NOT2._VP, OR1._VP, OR3._VP, SEL1._VP, SEL2._VP, SEL3._VP, XOR1._VP, XOR2._VP, XOR3._VP, XOR4._VP
- net GND: now also NAND1.V-, NOT1.V-, NOT2.V-, OR1.V-, OR3.V-, SEL1.V-, SEL2.V-, SEL3.V-, XOR1.V-, XOR2.V-, XOR3.V-, XOR4.V-; no longer NAND1._VN, NOT1._VN, NOT2._VN, OR1._VN, OR3._VN, SEL1._VN, SEL2._VN, SEL3._VN, XOR1._VN, XOR2._VN, XOR3._VN, XOR4._VN
Changed lines of the file:
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@@
 <?xml version="1.0" encoding="utf-8"?>
 <!DOCTYPE eagle SYSTEM "eagle.dtd">
-<eagle version="7.4.0">
+<eagle version="7.3.0">
 <drawing>
 <settings>
@@
 <instance part="GND6" gate="1" x="58.42" y="-99.06"/>
 <instance part="GND7" gate="1" x="129.54" y="-78.74"/>
-<instance part="CON2" gate="G$1" x="-20.32" y="-30.48"/>
+<instance part="CON2" gate="G$1" x="-20.32" y="-27.94"/>
 <instance part="GND8" gate="1" x="-10.16" y="-45.72"/>
 <instance part="P+8" gate="1" x="-7.62" y="-12.7"/>
@@
 <net name="+5V" class="0">
 <segment>
-<pinref part="XOR1" gate="G$1" pin="_VP"/>
+<pinref part="XOR1" gate="G$1" pin="V+"/>
 <pinref part="P+15" gate="1" pin="+5V"/>
 <wire x1="-12.7" y1="243.84" x2="-12.7" y2="241.3" width="0.1524" layer="91"/>
 </segment>
 <segment>
-<pinref part="XOR2" gate="G$1" pin="_VP"/>
+<pinref part="XOR2" gate="G$1" pin="V+"/>
 <pinref part="P+16" gate="1" pin="+5V"/>
 <wire x1="81.28" y1="261.62" x2="81.28" y2="259.08" width="0.1524" layer="91"/>
 </segment>
 <segment>
-<pinref part="NOT1" gate="G$1" pin="_VP"/>
+<pinref part="NOT1" gate="G$1" pin="V+"/>
 <pinref part="P+17" gate="1" pin="+5V"/>
 <wire x1="157.48" y1="198.12" x2="157.48" y2="195.58" width="0.1524" layer="91"/>
 </segment>
 <segment>
-<pinref part="XOR3" gate="G$1" pin="_VP"/>
+<pinref part="XOR3" gate="G$1" pin="V+"/>
 <pinref part="P+18" gate="1" pin="+5V"/>
 <wire x1="187.96" y1="276.86" x2="187.96" y2="279.4" width="0.1524" layer="91"/>
 </segment>
 <segment>
-<pinref part="OR1" gate="G$1" pin="_VP"/>
+<pinref part="OR1" gate="G$1" pin="V+"/>
 <pinref part="P+19" gate="1" pin="+5V"/>
 <wire x1="259.08" y1="238.76" x2="259.08" y2="236.22" width="0.1524" layer="91"/>
 </segment>
 <segment>
-<pinref part="OR3" gate="G$1" pin="_VP"/>
+<pinref part="OR3" gate="G$1" pin="V+"/>
 <pinref part="P+1" gate="1" pin="+5V"/>
 </segment>
 <segment>
-<pinref part="SEL2" gate="G$1" pin="_VP"/>
+<pinref part="SEL2" gate="G$1" pin="V+"/>
 <pinref part="P+2" gate="1" pin="+5V"/>
 <wire x1="66.04" y1="147.32" x2="66.04" y2="144.78" width="0.1524" layer="91"/>
 </segment>
 <segment>
-<pinref part="SEL1" gate="G$1" pin="_VP"/>
+<pinref part="SEL1" gate="G$1" pin="V+"/>
 <pinref part="P+3" gate="1" pin="+5V"/>
 <wire x1="-17.78" y1="78.74" x2="-17.78" y2="76.2" width="0.1524" layer="91"/>
 </segment>
 <segment>
-<pinref part="SEL3" gate="G$1" pin="_VP"/>
+<pinref part="SEL3" gate="G$1" pin="V+"/>
 <pinref part="P+4" gate="1" pin="+5V"/>
 <wire x1="144.78" y1="147.32" x2="144.78" y2="144.78" width="0.1524" layer="91"/>
 </segment>
 <segment>
-<pinref part="NOT2" gate="G$1" pin="_VP"/>
+<pinref part="NOT2" gate="G$1" pin="V+"/>
 <pinref part="P+5" gate="1" pin="+5V"/>
 <wire x1="25.4" y1="-53.34" x2="25.4" y2="-50.8" width="0.1524" layer="91"/>
 </segment>
 <segment>
-<pinref part="NAND1" gate="G$1" pin="_VP"/>
+<pinref part="NAND1" gate="G$1" pin="V+"/>
 <pinref part="P+6" gate="1" pin="+5V"/>
 <wire x1="58.42" y1="-58.42" x2="58.42" y2="-55.88" width="0.1524" layer="91"/>
 </segment>
 <segment>
-<pinref part="XOR4" gate="G$1" pin="_VP"/>
+<pinref part="XOR4" gate="G$1" pin="V+"/>
 <pinref part="P+7" gate="1" pin="+5V"/>
 <wire x1="129.54" y1="-12.7" x2="129.54" y2="-10.16" width="0.1524" layer="91"/>
@@
 <net name="GND" class="0">
 <segment>
-<pinref part="XOR1" gate="G$1" pin="_VN"/>
+<pinref part="XOR1" gate="G$1" pin="V-"/>
 <pinref part="GND15" gate="1" pin="GND"/>
 <wire x1="-12.7" y1="177.8" x2="-12.7" y2="180.34" width="0.1524" layer="91"/>
 </segment>
 <segment>
-<pinref part="XOR2" gate="G$1" pin="_VN"/>
+<pinref part="XOR2" gate="G$1" pin="V-"/>
 <pinref part="GND16" gate="1" pin="GND"/>
 <wire x1="81.28" y1="195.58" x2="81.28" y2="198.12" width="0.1524" layer="91"/>
 </segment>
 <segment>
-<pinref part="NOT1" gate="G$1" pin="_VN"/>
+<pinref part="NOT1" gate="G$1" pin="V-"/>
 <pinref part="GND17" gate="1" pin="GND"/>
 <wire x1="157.48" y1="167.64" x2="157.48" y2="170.18" width="0.1524" layer="91"/>
 </segment>
 <segment>
-<pinref part="XOR3" gate="G$1" pin="_VN"/>
+<pinref part="XOR3" gate="G$1" pin="V-"/>
 <pinref part="GND18" gate="1" pin="GND"/>
 <wire x1="187.96" y1="213.36" x2="187.96" y2="215.9" width="0.1524" layer="91"/>
 </segment>
 <segment>
-<pinref part="OR1" gate="G$1" pin="_VN"/>
+<pinref part="OR1" gate="G$1" pin="V-"/>
 <pinref part="GND19" gate="1" pin="GND"/>
 <wire x1="259.08" y1="177.8" x2="259.08" y2="180.34" width="0.1524" layer="91"/>
 </segment>
 <segment>
-<pinref part="OR3" gate="G$1" pin="_VN"/>
+<pinref part="OR3" gate="G$1" pin="V-"/>
 <pinref part="GND1" gate="1" pin="GND"/>
 </segment>
 <segment>
-<pinref part="SEL1" gate="G$1" pin="_VN"/>
+<pinref part="SEL1" gate="G$1" pin="V-"/>
 <pinref part="GND2" gate="1" pin="GND"/>
 <wire x1="-17.78" y1="5.08" x2="-17.78" y2="7.62" width="0.1524" layer="91"/>
 </segment>
 <segment>
-<pinref part="SEL2" gate="G$1" pin="_VN"/>
+<pinref part="SEL2" gate="G$1" pin="V-"/>
 <pinref part="GND3" gate="1" pin="GND"/>
 <wire x1="66.04" y1="-48.26" x2="66.04" y2="-45.72" width="0.1524" layer="91"/>
 </segment>
 <segment>
-<pinref part="SEL3" gate="G$1" pin="_VN"/>
+<pinref part="SEL3" gate="G$1" pin="V-"/>
 <pinref part="GND4" gate="1" pin="GND"/>
 <wire x1="144.78" y1="73.66" x2="144.78" y2="76.2" width="0.1524" layer="91"/>
 </segment>
 <segment>
-<pinref part="NOT2" gate="G$1" pin="_VN"/>
+<pinref part="NOT2" gate="G$1" pin="V-"/>
 <pinref part="GND5" gate="1" pin="GND"/>
 <wire x1="25.4" y1="-78.74" x2="25.4" y2="-81.28" width="0.1524" layer="91"/>
 </segment>
 <segment>
-<pinref part="NAND1" gate="G$1" pin="_VN"/>
+<pinref part="NAND1" gate="G$1" pin="V-"/>
 <pinref part="GND6" gate="1" pin="GND"/>
 <wire x1="58.42" y1="-93.98" x2="58.42" y2="-96.52" width="0.1524" layer="91"/>
 </segment>
 <segment>
-<pinref part="XOR4" gate="G$1" pin="_VN"/>
+<pinref part="XOR4" gate="G$1" pin="V-"/>
 <pinref part="GND7" gate="1" pin="GND"/>
 <wire x1="129.54" y1="-73.66" x2="129.54" y2="-76.2" width="0.1524" layer="91"/>

Commit message: Fixing stuff
Connections:
- net +5V: now also NAND1._VP, NOT1._VP, NOT2._VP, OR1._VP, OR3._VP, SEL1._VP, SEL2._VP, SEL3._VP, XOR1._VP, XOR2._VP, XOR3._VP, XOR4._VP; no longer NAND1.V+, NOT1.V+, NOT2.V+, OR1.V+, OR3.V+, SEL1.V+, SEL2.V+, SEL3.V+, XOR1.V+, XOR2.V+, XOR3.V+, XOR4.V+
- net GND: now also NAND1._VN, NOT1._VN, NOT2._VN, OR1._VN, OR3._VN, SEL1._VN, SEL2._VN, SEL3._VN, XOR1._VN, XOR2._VN, XOR3._VN, XOR4._VN; no longer NAND1.V-, NOT1.V-, NOT2.V-, OR1.V-, OR3.V-, SEL1.V-, SEL2.V-, SEL3.V-, XOR1.V-, XOR2.V-, XOR3.V-, XOR4.V-
Changed lines of the file:
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@@
 <net name="+5V" class="0">
 <segment>
-<pinref part="XOR1" gate="G$1" pin="V+"/>
+<pinref part="XOR1" gate="G$1" pin="_VP"/>
 <pinref part="P+15" gate="1" pin="+5V"/>
 <wire x1="-12.7" y1="243.84" x2="-12.7" y2="241.3" width="0.1524" layer="91"/>
 </segment>
 <segment>
-<pinref part="XOR2" gate="G$1" pin="V+"/>
+<pinref part="XOR2" gate="G$1" pin="_VP"/>
 <pinref part="P+16" gate="1" pin="+5V"/>
 <wire x1="81.28" y1="261.62" x2="81.28" y2="259.08" width="0.1524" layer="91"/>
 </segment>
 <segment>
-<pinref part="NOT1" gate="G$1" pin="V+"/>
+<pinref part="NOT1" gate="G$1" pin="_VP"/>
 <pinref part="P+17" gate="1" pin="+5V"/>
 <wire x1="157.48" y1="198.12" x2="157.48" y2="195.58" width="0.1524" layer="91"/>
 </segment>
 <segment>
-<pinref part="XOR3" gate="G$1" pin="V+"/>
+<pinref part="XOR3" gate="G$1" pin="_VP"/>
 <pinref part="P+18" gate="1" pin="+5V"/>
 <wire x1="187.96" y1="276.86" x2="187.96" y2="279.4" width="0.1524" layer="91"/>
 </segment>
 <segment>
-<pinref part="OR1" gate="G$1" pin="V+"/>
+<pinref part="OR1" gate="G$1" pin="_VP"/>
 <pinref part="P+19" gate="1" pin="+5V"/>
 <wire x1="259.08" y1="238.76" x2="259.08" y2="236.22" width="0.1524" layer="91"/>
 </segment>
 <segment>
-<pinref part="OR3" gate="G$1" pin="V+"/>
+<pinref part="OR3" gate="G$1" pin="_VP"/>
 <pinref part="P+1" gate="1" pin="+5V"/>
 </segment>
 <segment>
-<pinref part="SEL2" gate="G$1" pin="V+"/>
+<pinref part="SEL2" gate="G$1" pin="_VP"/>
 <pinref part="P+2" gate="1" pin="+5V"/>
 <wire x1="66.04" y1="147.32" x2="66.04" y2="144.78" width="0.1524" layer="91"/>
 </segment>
 <segment>
-<pinref part="SEL1" gate="G$1" pin="V+"/>
+<pinref part="SEL1" gate="G$1" pin="_VP"/>
 <pinref part="P+3" gate="1" pin="+5V"/>
 <wire x1="-17.78" y1="78.74" x2="-17.78" y2="76.2" width="0.1524" layer="91"/>
 </segment>
 <segment>
-<pinref part="SEL3" gate="G$1" pin="V+"/>
+<pinref part="SEL3" gate="G$1" pin="_VP"/>
 <pinref part="P+4" gate="1" pin="+5V"/>
 <wire x1="144.78" y1="147.32" x2="144.78" y2="144.78" width="0.1524" layer="91"/>
 </segment>
 <segment>
-<pinref part="NOT2" gate="G$1" pin="V+"/>
+<pinref part="NOT2" gate="G$1" pin="_VP"/>
 <pinref part="P+5" gate="1" pin="+5V"/>
 <wire x1="25.4" y1="-53.34" x2="25.4" y2="-50.8" width="0.1524" layer="91"/>
 </segment>
 <segment>
-<pinref part="NAND1" gate="G$1" pin="V+"/>
+<pinref part="NAND1" gate="G$1" pin="_VP"/>
 <pinref part="P+6" gate="1" pin="+5V"/>
 <wire x1="58.42" y1="-58.42" x2="58.42" y2="-55.88" width="0.1524" layer="91"/>
 </segment>
 <segment>
-<pinref part="XOR4" gate="G$1" pin="V+"/>
+<pinref part="XOR4" gate="G$1" pin="_VP"/>
 <pinref part="P+7" gate="1" pin="+5V"/>
 <wire x1="129.54" y1="-12.7" x2="129.54" y2="-10.16" width="0.1524" layer="91"/>
@@
 <net name="GND" class="0">
 <segment>
-<pinref part="XOR1" gate="G$1" pin="V-"/>
+<pinref part="XOR1" gate="G$1" pin="_VN"/>
 <pinref part="GND15" gate="1" pin="GND"/>
 <wire x1="-12.7" y1="177.8" x2="-12.7" y2="180.34" width="0.1524" layer="91"/>
 </segment>
 <segment>
-<pinref part="XOR2" gate="G$1" pin="V-"/>
+<pinref part="XOR2" gate="G$1" pin="_VN"/>
 <pinref part="GND16" gate="1" pin="GND"/>
 <wire x1="81.28" y1="195.58" x2="81.28" y2="198.12" width="0.1524" layer="91"/>
 </segment>
 <segment>
-<pinref part="NOT1" gate="G$1" pin="V-"/>
+<pinref part="NOT1" gate="G$1" pin="_VN"/>
 <pinref part="GND17" gate="1" pin="GND"/>
 <wire x1="157.48" y1="167.64" x2="157.48" y2="170.18" width="0.1524" layer="91"/>
 </segment>
 <segment>
-<pinref part="XOR3" gate="G$1" pin="V-"/>
+<pinref part="XOR3" gate="G$1" pin="_VN"/>
 <pinref part="GND18" gate="1" pin="GND"/>
 <wire x1="187.96" y1="213.36" x2="187.96" y2="215.9" width="0.1524" layer="91"/>
 </segment>
 <segment>
-<pinref part="OR1" gate="G$1" pin="V-"/>
+<pinref part="OR1" gate="G$1" pin="_VN"/>
 <pinref part="GND19" gate="1" pin="GND"/>
 <wire x1="259.08" y1="177.8" x2="259.08" y2="180.34" width="0.1524" layer="91"/>
 </segment>
 <segment>
-<pinref part="OR3" gate="G$1" pin="V-"/>
+<pinref part="OR3" gate="G$1" pin="_VN"/>
 <pinref part="GND1" gate="1" pin="GND"/>
 </segment>
 <segment>
-<pinref part="SEL1" gate="G$1" pin="V-"/>
+<pinref part="SEL1" gate="G$1" pin="_VN"/>
 <pinref part="GND2" gate="1" pin="GND"/>
 <wire x1="-17.78" y1="5.08" x2="-17.78" y2="7.62" width="0.1524" layer="91"/>
 </segment>
 <segment>
-<pinref part="SEL2" gate="G$1" pin="V-"/>
+<pinref part="SEL2" gate="G$1" pin="_VN"/>
 <pinref part="GND3" gate="1" pin="GND"/>
 <wire x1="66.04" y1="-48.26" x2="66.04" y2="-45.72" width="0.1524" layer="91"/>
 </segment>
 <segment>
-<pinref part="SEL3" gate="G$1" pin="V-"/>
+<pinref part="SEL3" gate="G$1" pin="_VN"/>
 <pinref part="GND4" gate="1" pin="GND"/>
 <wire x1="144.78" y1="73.66" x2="144.78" y2="76.2" width="0.1524" layer="91"/>
 </segment>
 <segment>
-<pinref part="NOT2" gate="G$1" pin="V-"/>
+<pinref part="NOT2" gate="G$1" pin="_VN"/>
 <pinref part="GND5" gate="1" pin="GND"/>
 <wire x1="25.4" y1="-78.74" x2="25.4" y2="-81.28" width="0.1524" layer="91"/>
 </segment>
 <segment>
-<pinref part="NAND1" gate="G$1" pin="V-"/>
+<pinref part="NAND1" gate="G$1" pin="_VN"/>
 <pinref part="GND6" gate="1" pin="GND"/>
 <wire x1="58.42" y1="-93.98" x2="58.42" y2="-96.52" width="0.1524" layer="91"/>
 </segment>
 <segment>
-<pinref part="XOR4" gate="G$1" pin="V-"/>
+<pinref part="XOR4" gate="G$1" pin="_VN"/>
 <pinref part="GND7" gate="1" pin="GND"/>
 <wire x1="129.54" y1="-73.66" x2="129.54" y2="-76.2" width="0.1524" layer="91"/>

Commit message: reordering board
Connections:
- net +5V: now also CON2.19; no longer CON2.2
- net A: now also CON2.10, SEL2.I4; no longer CON2.1, SEL2.I1
- net B: now also SEL2.I2; no longer SEL2.I8
- net CARRY: now also CON2.11; no longer CON2.15
- net EQUAL_IN: now also CON2.13; no longer CON2.9
- net EQUAL_OUT: now also CON2.17; no longer CON2.19
- net LEFT_IN: now also CON2.7, SEL2.I3; no longer CON2.5, SEL2.I7
- net N$2: now also SEL2.I1; no longer SEL2.I6
- net NAND: now also SEL2.I8; no longer SEL2.I2
- net NOR: now also SEL2.I7; no longer SEL2.I3
- net OVERFLOW: now also CON2.5; no longer CON2.17
- net RESULT: now also CON2.15; no longer CON2.11
- net RIGHT_IN: now also CON2.1; no longer CON2.7
- net RIGHT_OUT: now also CON2.9; no longer CON2.13
- net S_AND: now also CON2.18, SEL2.S8; no longer CON2.6, SEL2.S2
- net S_CMP: now also CON2.6, SEL2.S3; no longer CON2.16, SEL2.S7
- net S_ID: now also CON2.8, SEL2.S4; no longer CON2.4, SEL2.S1
- net S_LOAD: now also CON2.4, SEL2.S2; no longer CON2.18, SEL2.S8
- net S_NOR: now also CON2.16, SEL2.S7; no longer CON2.8, SEL2.S3
- net S_SHIFT: now also CON2.2, SEL2.S1; no longer CON2.14, SEL2.S6
- net S_XOR: now also CON2.14, SEL2.S6; no longer CON2.10, SEL2.S4
- net XOR: now also SEL2.I6; no longer SEL2.I4

Commit message: Basic cleanups
Other:
- moved on the sheet: SEL1

Commit message: Naming cleanup
Connections:
- net CARRY renamed CARRY_OUT
- net INV_ADD renamed INVERT
Changed lines of the file:
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@@
 </segment>
 </net>
-<net name="CARRY" class="0">
+<net name="CARRY_OUT" class="0">
 <segment>
 <pinref part="XOR3" gate="G$1" pin="XOR"/>
@@
 </segment>
 </net>
-<net name="INV_ADD" class="0">
+<net name="INVERT" class="0">
 <segment>
 <pinref part="XOR1" gate="G$1" pin="B"/>
