File: hw/composites/alu_slice.brd (EAGLE design)
At the start: 50 x 50 mm, 6 parts, among them CON2 GENERIC-2X10

Commit message: adds substraction
Parts:
- added XOR4: XOR, p.peter-gator:XOR
Connections:
- new net N$2: XOR2.B, XOR4.XOR
- new net SUBTRACT: CON2.9, XOR4.B
- net +5V: now also CON2.2, XOR4._VP; no longer CON2.19
- net B: now also XOR4.A; no longer XOR2.B
- net GND: now also XOR4._VN
- net NC: now also CON2.15; no longer CON2.8, CON2.9
- net RESULT: now also CON2.19; no longer CON2.15
- net S_ADD: now also CON2.8; no longer CON2.6
- net S_AND: now also CON2.6; no longer CON2.4
- net S_ID: now also CON2.4; no longer CON2.2
Changed lines of the file:
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@@
 <element name="CON2" library="p.peter-connectors" package="PINHEADER-100MIL-2X10-EDGE" value="GENERIC-2X10" x="28.5" y="0"/>
 <element name="XOR1" library="p.peter-gator" package="XOR" value="XOR" x="0.5" y="-20"/>
+<element name="XOR4" library="p.peter-gator" package="XOR" value="XOR" x="0" y="-34"/>
 </elements>
 <signals>
@@
 <contactref element="OR1" pad="_VP"/>
 <contactref element="SEL2" pad="_VP"/>
-<contactref element="CON2" pad="19"/>
+<contactref element="CON2" pad="2"/>
 <contactref element="XOR1" pad="_VP"/>
+<contactref element="XOR4" pad="_VP"/>
 <wire x1="37.5" y1="34.5" x2="48.5" y2="32" width="0" layer="19" extent="1-1"/>
 <wire x1="15.5" y1="32" x2="37.5" y2="34.5" width="0" layer="19" extent="1-1"/>
 <wire x1="48" y1="5" x2="48.5" y2="32" width="0" layer="19" extent="1-1"/>
-<wire x1="39.93" y1="1.27" x2="48" y2="5" width="0" layer="19" extent="1-16"/>
-<wire x1="1.5" y1="-7.5" x2="39.93" y2="1.27" width="0" layer="19" extent="1-16"/>
+<wire x1="17.07" y1="1.27" x2="48" y2="5" width="0" layer="19" extent="1-16"/>
+<wire x1="1.5" y1="-7.5" x2="17.07" y2="1.27" width="0" layer="19" extent="1-16"/>
+<wire x1="1" y1="-21.5" x2="1.5" y2="-7.5" width="0" layer="19" extent="1-1"/>
 </signal>
 <signal name="GND">
@@
 <contactref element="CON2" pad="20"/>
 <contactref element="XOR1" pad="_VN"/>
+<contactref element="XOR4" pad="_VN"/>
 <wire x1="27.8" y1="32" x2="47.5" y2="32" width="0" layer="19" extent="1-1"/>
 <wire x1="25.2" y1="34.5" x2="27.8" y2="32" width="0" layer="19" extent="1-1"/>
@@
 <wire x1="39.93" y1="1.27" x2="46" y2="5" width="0" layer="19" extent="1-1"/>
 <wire x1="13.8" y1="-7.5" x2="39.93" y2="1.27" width="0" layer="19" extent="1-1"/>
+<wire x1="13.3" y1="-21.5" x2="13.8" y2="-7.5" width="0" layer="19" extent="1-1"/>
 </signal>
 <signal name="NOR">
@@
 <contactref element="SEL2" pad="I2"/>
 <contactref element="CON2" pad="3"/>
-<contactref element="XOR2" pad="B"/>
-<wire x1="17.8" y1="5" x2="38" y2="47" width="0" layer="19" extent="1-1"/>
-<wire x1="19.61" y1="1.27" x2="17.8" y2="5" width="0" layer="19" extent="1-16"/>
+<contactref element="XOR4" pad="A"/>
+<wire x1="19.61" y1="1.27" x2="12.5" y2="-34" width="0" layer="19" extent="1-16"/>
+<wire x1="17.8" y1="5" x2="19.61" y2="1.27" width="0" layer="19" extent="1-16"/>
 </signal>
 <signal name="LEFT_IN">
@@
 <signal name="S_ADD">
 <contactref element="SEL2" pad="S5"/>
-<contactref element="CON2" pad="6"/>
-<wire x1="22.15" y1="1.27" x2="28.8" y2="5" width="0" layer="19" extent="1-1"/>
+<contactref element="CON2" pad="8"/>
+<wire x1="24.69" y1="1.27" x2="28.8" y2="5" width="0" layer="19" extent="1-1"/>
 </signal>
 <signal name="S_CMP">
@@
 <signal name="S_ID">
 <contactref element="SEL2" pad="S4"/>
-<contactref element="CON2" pad="2"/>
-<wire x1="17.07" y1="1.27" x2="24.4" y2="5" width="0" layer="19" extent="1-1"/>
+<contactref element="CON2" pad="4"/>
+<wire x1="19.61" y1="1.27" x2="24.4" y2="5" width="0" layer="19" extent="1-1"/>
 </signal>
 <signal name="S_AND">
 <contactref element="SEL2" pad="S8"/>
-<contactref element="CON2" pad="4"/>
-<wire x1="19.61" y1="1.27" x2="42" y2="5" width="0" layer="19" extent="1-1"/>
+<contactref element="CON2" pad="6"/>
+<wire x1="22.15" y1="1.27" x2="42" y2="5" width="0" layer="19" extent="1-1"/>
 </signal>
 <signal name="S_SHIFT">
@@
 </signal>
 <signal name="RESULT">
-<contactref element="CON2" pad="15"/>
+<contactref element="CON2" pad="19"/>
 <contactref element="XOR1" pad="XOR"/>
-<wire x1="11" y1="-7.5" x2="34.85" y2="1.27" width="0" layer="19" extent="1-16"/>
+<wire x1="11" y1="-7.5" x2="39.93" y2="1.27" width="0" layer="19" extent="1-16"/>
 </signal>
 <signal name="N$4">
 </signal>
 <signal name="NC">
-<contactref element="CON2" pad="9"/>
 <contactref element="CON2" pad="11"/>
 <contactref element="CON2" pad="13"/>
-<contactref element="CON2" pad="8"/>
+<contactref element="CON2" pad="15"/>
 <contactref element="CON2" pad="10"/>
 <contactref element="CON2" pad="12"/>
@@
 <wire x1="29.77" y1="1.27" x2="32.31" y2="1.27" width="0" layer="19" extent="16-16"/>
 <wire x1="29.77" y1="1.27" x2="29.77" y2="1.27" width="0" layer="19" extent="1-16"/>
-<wire x1="27.23" y1="1.27" x2="29.77" y2="1.27" width="0" layer="19" extent="16-16"/>
-<wire x1="27.23" y1="1.27" x2="27.23" y2="1.27" width="0" layer="19" extent="1-16"/>
-<wire x1="24.69" y1="1.27" x2="27.23" y2="1.27" width="0" layer="19" extent="1-16"/>
+<wire x1="27.23" y1="1.27" x2="29.77" y2="1.27" width="0" layer="19" extent="1-16"/>
+<wire x1="34.85" y1="1.27" x2="27.23" y2="1.27" width="0" layer="19" extent="1-1"/>
 </signal>
 <signal name="INVERT_OUT">
@@
 <wire x1="13" y1="-20" x2="47" y2="5" width="0" layer="19" extent="1-1"/>
 </signal>
+<signal name="N$2">
+<contactref element="XOR2" pad="B"/>
+<contactref element="XOR4" pad="XOR"/>
+<wire x1="10.5" y1="-21.5" x2="38" y2="47" width="0" layer="19" extent="1-1"/>
+</signal>
+<signal name="SUBTRACT">
+<contactref element="XOR4" pad="B"/>
+<contactref element="CON2" pad="9"/>
+<wire x1="27.23" y1="1.27" x2="0.5" y2="-34" width="0" layer="19" extent="1-16"/>
+</signal>
 </signals>
