File: hw/singleGates/minimal/1-BitSelect.brd (EAGLE design)
At the start: 15 parts, among them Q1 BC817, Q2 BC817, Q3 BC817, Q4 BC817, Q5 BC817, Q6 BC817

Commit message: Add led output and prepare first alu slice
Parts:
- R1, R4, R9: device p.peter-gator:R0603 -> p.peter-rcl:R0603-MARK
Changed lines of the file:
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@@
 <grid distance="0.1" unitdist="mm" unit="mm" style="lines" multiple="1" display="yes" altdistance="0.05" altunitdist="mm" altunit="mm"/>
 <layers>
-<layer number="1" name="Top" color="4" fill="1" visible="yes" active="yes"/>
+<layer number="1" name="Top" color="4" fill="1" visible="no" active="yes"/>
 <layer number="16" name="Bottom" color="1" fill="1" visible="yes" active="yes"/>
 <layer number="17" name="Pads" color="2" fill="1" visible="yes" active="yes"/>
 <layer number="18" name="Vias" color="2" fill="1" visible="yes" active="yes"/>
-<layer number="19" name="Unrouted" color="6" fill="1" visible="yes" active="yes"/>
+<layer number="19" name="Unrouted" color="6" fill="1" visible="no" active="yes"/>
 <layer number="20" name="Dimension" color="15" fill="1" visible="yes" active="yes"/>
 <layer number="21" name="tPlace" color="7" fill="1" visible="yes" active="yes"/>
-<layer number="22" name="bPlace" color="7" fill="1" visible="yes" active="yes"/>
-<layer number="23" name="tOrigins" color="15" fill="1" visible="yes" active="yes"/>
-<layer number="24" name="bOrigins" color="15" fill="1" visible="yes" active="yes"/>
-<layer number="25" name="tNames" color="7" fill="1" visible="no" active="yes"/>
+<layer number="22" name="bPlace" color="7" fill="1" visible="no" active="yes"/>
+<layer number="23" name="tOrigins" color="15" fill="1" visible="no" active="yes"/>
+<layer number="24" name="bOrigins" color="15" fill="1" visible="no" active="yes"/>
+<layer number="25" name="tNames" color="7" fill="1" visible="yes" active="yes"/>
 <layer number="26" name="bNames" color="7" fill="1" visible="no" active="yes"/>
-<layer number="27" name="tValues" color="7" fill="1" visible="no" active="yes"/>
+<layer number="27" name="tValues" color="7" fill="1" visible="yes" active="yes"/>
 <layer number="28" name="bValues" color="7" fill="1" visible="no" active="yes"/>
-<layer number="29" name="tStop" color="7" fill="3" visible="no" active="yes"/>
+<layer number="29" name="tStop" color="7" fill="3" visible="yes" active="yes"/>
 <layer number="30" name="bStop" color="7" fill="6" visible="no" active="yes"/>
 <layer number="31" name="tCream" color="7" fill="4" visible="no" active="yes"/>
@@
 <layer number="37" name="tTest" color="7" fill="1" visible="no" active="yes"/>
 <layer number="38" name="bTest" color="7" fill="1" visible="no" active="yes"/>
-<layer number="39" name="tKeepout" color="4" fill="11" visible="yes" active="yes"/>
-<layer number="40" name="bKeepout" color="1" fill="11" visible="yes" active="yes"/>
-<layer number="41" name="tRestrict" color="4" fill="10" visible="yes" active="yes"/>
-<layer number="42" name="bRestrict" color="1" fill="10" visible="yes" active="yes"/>
+<layer number="39" name="tKeepout" color="4" fill="11" visible="no" active="yes"/>
+<layer number="40" name="bKeepout" color="1" fill="11" visible="no" active="yes"/>
+<layer number="41" name="tRestrict" color="4" fill="10" visible="no" active="yes"/>
+<layer number="42" name="bRestrict" color="1" fill="10" visible="no" active="yes"/>
 <layer number="43" name="vRestrict" color="2" fill="10" visible="no" active="yes"/>
 <layer number="44" name="Drills" color="7" fill="1" visible="no" active="yes"/>
@@
 <layer number="110" name="fp0" color="7" fill="1" visible="no" active="yes"/>
 <layer number="116" name="Patch_BOT" color="9" fill="4" visible="no" active="yes"/>
-<layer number="121" name="_tsilk" color="7" fill="1" visible="no" active="yes"/>
+<layer number="121" name="_tsilk" color="7" fill="1" visible="yes" active="yes"/>
 <layer number="122" name="_bsilk" color="7" fill="1" visible="no" active="yes"/>
 <layer number="123" name="tTestmark" color="7" fill="1" visible="no" active="yes"/>
@@
 <attribute name="SV_SPICE_PREFIX" value="R" x="1" y="4.9" size="1.778" layer="27" rot="R90" display="off"/>
 </element>
-<element name="R1" library="p.peter-gator" package="R0603" value="1k" x="10.1" y="12.8" smashed="yes">
-<attribute name="SV_SPICE_ORDER" value="1;2" x="10.1" y="12.8" size="1.778" layer="27" display="off"/>
-<attribute name="SV_SPICE_PREFIX" value="R" x="10.1" y="12.8" size="1.778" layer="27" display="off"/>
-</element>
+<element name="R1" library="p.peter-rcl" package="R0603-MARK" value="1k" x="10.1" y="12.8" smashed="yes"/>
 <element name="R6" library="p.peter-gator" package="R0603" value="10k" x="7.6" y="4.9" smashed="yes" rot="R90">
 <attribute name="SV_SPICE_ORDER" value="1;2" x="7.6" y="4.9" size="1.778" layer="27" rot="R90" display="off"/>
@@
 <attribute name="SV_SPICE_PREFIX" value="R" x="5.5" y="4.9" size="1.778" layer="27" rot="R90" display="off"/>
 </element>
-<element name="R9" library="p.peter-gator" package="R0603" value="1k" x="10.3" y="4.5" smashed="yes">
-<attribute name="SV_SPICE_ORDER" value="1;2" x="10.3" y="4.5" size="1.778" layer="27" display="off"/>
-<attribute name="SV_SPICE_PREFIX" value="R" x="10.3" y="4.5" size="1.778" layer="27" display="off"/>
-</element>
+<element name="R9" library="p.peter-rcl" package="R0603-MARK" value="1k" x="10.3" y="4.5" smashed="yes"/>
 <element name="R8" library="p.peter-gator" package="R0603" value="10k" x="10.1" y="10.6" smashed="yes">
 <attribute name="SV_SPICE_ORDER" value="1;2" x="10.1" y="10.6" size="1.778" layer="27" display="off"/>
 <attribute name="SV_SPICE_PREFIX" value="R" x="10.1" y="10.6" size="1.778" layer="27" display="off"/>
 </element>
-<element name="R4" library="p.peter-gator" package="R0603" value="1k" x="10.3" y="2.3" smashed="yes">
-<attribute name="SV_SPICE_ORDER" value="1;2" x="10.3" y="2.3" size="1.778" layer="27" display="off"/>
-<attribute name="SV_SPICE_PREFIX" value="R" x="10.3" y="2.3" size="1.778" layer="27" display="off"/>
-</element>
+<element name="R4" library="p.peter-rcl" package="R0603-MARK" value="1k" x="10.3" y="2.3" smashed="yes"/>
 <element name="R5" library="p.peter-gator" package="R0603" value="10k" x="3.2" y="1.7" smashed="yes" rot="R270">
 <attribute name="SV_SPICE_ORDER" value="1;2" x="3.2" y="1.7" size="1.778" layer="27" rot="R270" display="off"/>
