File: hw/singleGates/minimal/XOR.brd (EAGLE design)
At the start: 15 parts, among them Q1 BC817, Q2 BC817, Q3 BC817, Q4 BC817, Q5 BC817, Q6 BC817

Commit message: Add led output and prepare first alu slice
Parts:
- R3, R6, R9: device p.peter-gator:R0603 -> p.peter-rcl:R0603-MARK
Changed lines of the file:
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@@
 <grid distance="0.1" unitdist="mm" unit="mm" style="lines" multiple="1" display="yes" altdistance="0.05" altunitdist="mm" altunit="mm"/>
 <layers>
-<layer number="1" name="Top" color="4" fill="1" visible="yes" active="yes"/>
-<layer number="16" name="Bottom" color="1" fill="1" visible="yes" active="yes"/>
+<layer number="1" name="Top" color="4" fill="1" visible="no" active="yes"/>
+<layer number="16" name="Bottom" color="1" fill="1" visible="no" active="yes"/>
 <layer number="17" name="Pads" color="2" fill="1" visible="yes" active="yes"/>
 <layer number="18" name="Vias" color="2" fill="1" visible="yes" active="yes"/>
-<layer number="19" name="Unrouted" color="6" fill="1" visible="yes" active="yes"/>
+<layer number="19" name="Unrouted" color="6" fill="1" visible="no" active="yes"/>
 <layer number="20" name="Dimension" color="15" fill="1" visible="yes" active="yes"/>
 <layer number="21" name="tPlace" color="7" fill="1" visible="yes" active="yes"/>
-<layer number="22" name="bPlace" color="7" fill="1" visible="yes" active="yes"/>
-<layer number="23" name="tOrigins" color="15" fill="1" visible="yes" active="yes"/>
-<layer number="24" name="bOrigins" color="15" fill="1" visible="yes" active="yes"/>
+<layer number="22" name="bPlace" color="7" fill="1" visible="no" active="yes"/>
+<layer number="23" name="tOrigins" color="15" fill="1" visible="no" active="yes"/>
+<layer number="24" name="bOrigins" color="15" fill="1" visible="no" active="yes"/>
 <layer number="25" name="tNames" color="7" fill="1" visible="yes" active="yes"/>
-<layer number="26" name="bNames" color="7" fill="1" visible="yes" active="yes"/>
+<layer number="26" name="bNames" color="7" fill="1" visible="no" active="yes"/>
 <layer number="27" name="tValues" color="7" fill="1" visible="yes" active="yes"/>
-<layer number="28" name="bValues" color="7" fill="1" visible="yes" active="yes"/>
-<layer number="29" name="tStop" color="7" fill="3" visible="no" active="yes"/>
+<layer number="28" name="bValues" color="7" fill="1" visible="no" active="yes"/>
+<layer number="29" name="tStop" color="7" fill="3" visible="yes" active="yes"/>
 <layer number="30" name="bStop" color="7" fill="6" visible="no" active="yes"/>
 <layer number="31" name="tCream" color="7" fill="4" visible="no" active="yes"/>
@@
 <layer number="37" name="tTest" color="7" fill="1" visible="no" active="yes"/>
 <layer number="38" name="bTest" color="7" fill="1" visible="no" active="yes"/>
-<layer number="39" name="tKeepout" color="4" fill="11" visible="yes" active="yes"/>
-<layer number="40" name="bKeepout" color="1" fill="11" visible="yes" active="yes"/>
-<layer number="41" name="tRestrict" color="4" fill="10" visible="yes" active="yes"/>
-<layer number="42" name="bRestrict" color="1" fill="10" visible="yes" active="yes"/>
-<layer number="43" name="vRestrict" color="2" fill="10" visible="yes" active="yes"/>
+<layer number="39" name="tKeepout" color="4" fill="11" visible="no" active="yes"/>
+<layer number="40" name="bKeepout" color="1" fill="11" visible="no" active="yes"/>
+<layer number="41" name="tRestrict" color="4" fill="10" visible="no" active="yes"/>
+<layer number="42" name="bRestrict" color="1" fill="10" visible="no" active="yes"/>
+<layer number="43" name="vRestrict" color="2" fill="10" visible="no" active="yes"/>
 <layer number="44" name="Drills" color="7" fill="1" visible="no" active="yes"/>
 <layer number="45" name="Holes" color="7" fill="1" visible="no" active="yes"/>
 <layer number="46" name="Milling" color="3" fill="1" visible="no" active="yes"/>
 <layer number="47" name="Measures" color="7" fill="1" visible="no" active="yes"/>
-<layer number="48" name="Document" color="7" fill="1" visible="yes" active="yes"/>
-<layer number="49" name="Reference" color="7" fill="1" visible="yes" active="yes"/>
+<layer number="48" name="Document" color="7" fill="1" visible="no" active="yes"/>
+<layer number="49" name="Reference" color="7" fill="1" visible="no" active="yes"/>
 <layer number="50" name="dxf" color="7" fill="1" visible="no" active="no"/>
-<layer number="51" name="tDocu" color="7" fill="1" visible="yes" active="yes"/>
-<layer number="52" name="bDocu" color="7" fill="1" visible="yes" active="yes"/>
+<layer number="51" name="tDocu" color="7" fill="1" visible="no" active="yes"/>
+<layer number="52" name="bDocu" color="7" fill="1" visible="no" active="yes"/>
 <layer number="53" name="tGND_GNDA" color="7" fill="9" visible="no" active="no"/>
 <layer number="54" name="bGND_GNDA" color="1" fill="9" visible="no" active="no"/>
@@
 <layer number="110" name="fp0" color="7" fill="1" visible="no" active="yes"/>
 <layer number="116" name="Patch_BOT" color="9" fill="4" visible="no" active="yes"/>
-<layer number="121" name="_tsilk" color="7" fill="1" visible="no" active="yes"/>
+<layer number="121" name="_tsilk" color="7" fill="1" visible="yes" active="yes"/>
 <layer number="122" name="_bsilk" color="7" fill="1" visible="no" active="yes"/>
 <layer number="123" name="tTestmark" color="7" fill="1" visible="no" active="yes"/>
@@
 <wire x1="14" y1="12.5" x2="0" y2="12.5" width="0.2" layer="22" style="shortdash"/>
 <wire x1="0" y1="12.5" x2="0" y2="0" width="0.2" layer="22" style="shortdash"/>
-<wire x1="5.3" y1="11.7" x2="5.3" y2="10.9" width="0.4" layer="21"/>
-<wire x1="2.1" y1="8.8" x2="2.1" y2="9.6" width="0.4" layer="21"/>
-<wire x1="7.8" y1="2.4" x2="8.6" y2="2.4" width="0.4" layer="21"/>
 </plain>
 <attributes>
@@
 <attribute name="SV_SPICE_PREFIX" value="R" x="5.8" y="2.4" size="1.778" layer="27" rot="R90" display="off"/>
 </element>
-<element name="R3" library="p.peter-gator" package="R0603" value="1k" x="8.2" y="2.4" smashed="yes" rot="R90">
-<attribute name="SV_SPICE_ORDER" value="1;2" x="8.2" y="2.4" size="1.778" layer="27" rot="R90" display="off"/>
-<attribute name="SV_SPICE_PREFIX" value="R" x="8.2" y="2.4" size="1.778" layer="27" rot="R90" display="off"/>
-</element>
-<element name="R6" library="p.peter-gator" package="R0603" value="1k" x="2.1" y="9.2" smashed="yes" rot="R180">
-<attribute name="SV_SPICE_ORDER" value="1;2" x="2.1" y="9.2" size="1.778" layer="27" rot="R180" display="off"/>
-<attribute name="SV_SPICE_PREFIX" value="R" x="2.1" y="9.2" size="1.778" layer="27" rot="R180" display="off"/>
-</element>
-<element name="R9" library="p.peter-gator" package="R0603" value="1k" x="5.3" y="11.3" smashed="yes" rot="R180">
-<attribute name="SV_SPICE_ORDER" value="1;2" x="5.3" y="11.3" size="1.778" layer="27" rot="R180" display="off"/>
-<attribute name="SV_SPICE_PREFIX" value="R" x="5.3" y="11.3" size="1.778" layer="27" rot="R180" display="off"/>
-</element>
+<element name="R3" library="p.peter-rcl" package="R0603-MARK" value="1k" x="8.2" y="2.4" smashed="yes" rot="R90"/>
+<element name="R6" library="p.peter-rcl" package="R0603-MARK" value="1k" x="2.1" y="9.2" smashed="yes" rot="R180"/>
+<element name="R9" library="p.peter-rcl" package="R0603-MARK" value="1k" x="5.3" y="11.3" smashed="yes" rot="R180"/>
 <element name="Q1" library="p.peter-gator" package="SOT23" value="BC817" x="1.8" y="6.2" smashed="yes">
 <attribute name="SV_SPICE_MODEL" value="NPN ()" x="1.8" y="6.2" size="1.778" layer="27" display="off"/>
