File: hw/singleGates/minimal/XOR.sch (EAGLE design)
At the start: 15 parts, among them Q1 BC817, Q2 BC817, Q3 BC817, Q4 BC817, Q5 BC817, Q6 BC817

Commit message: Add led output and prepare first alu slice
Parts:
- R3, R6, R9: device p.peter-gator:R-EU_R0603 -> p.peter-rcl:R-EU-MARKEDR0603
Changed lines of the file:
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@@
 <part name="R7" library="p.peter-gator" deviceset="R-EU_" device="R0603" value="10k"/>
 <part name="R8" library="p.peter-gator" deviceset="R-EU_" device="R0603" value="10k"/>
-<part name="R3" library="p.peter-gator" deviceset="R-EU_" device="R0603" value="1k"/>
-<part name="R6" library="p.peter-gator" deviceset="R-EU_" device="R0603" value="1k"/>
-<part name="R9" library="p.peter-gator" deviceset="R-EU_" device="R0603" value="1k"/>
+<part name="R3" library="p.peter-rcl" deviceset="R-EU-MARKED" device="R0603" value="1k"/>
+<part name="R6" library="p.peter-rcl" deviceset="R-EU-MARKED" device="R0603" value="1k"/>
+<part name="R9" library="p.peter-rcl" deviceset="R-EU-MARKED" device="R0603" value="1k"/>
 <part name="Q1" library="p.peter-gator" deviceset="TRANSISTOR-NPN-GENERIC" device="-SOT23-BEC" technology="DEFAULT" value="BC817"/>
 <part name="Q2" library="p.peter-gator" deviceset="TRANSISTOR-NPN-GENERIC" device="-SOT23-BEC" technology="DEFAULT" value="BC817"/>
